File: blackwing.kicad_pcb (KiCad board)
At the start: 2 copper layers, 161.9 x 123.8 mm, 36 parts, among them J1 Conn_01x04, SW00 SW_Push, SW01 SW_Push, SW02 SW_Push, SW03 SW_Push, SW04 SW_Push, SW05 SW_Push, SW10 SW_Push, SW11 SW_Push, SW12 SW_Push, SW13 SW_Push, SW14 SW_Push, SW15 SW_Push, SW20 SW_Push, SW21 SW_Push, SW22 SW_Push, SW23 SW_Push, SW24 SW_Push, SW25 SW_Push, SW30 SW_Push, SW31 SW_Push, SW32 SW_Push, SW33 SW_Push, SW34 SW_Push, SW35 SW_Push, SW40 SW_Push, SW41 SW_Push, SW42 SW_Push, SW43 SW_Push, SW44 SW_Push, SW45 SW_Push, SW50 SW_Push, U1 CORE51822, U2 CORE51822

Commit message: v 2.1
Parts:
- moved SW01 7.14 mm to (50.8, 10.2)
- moved SW12 4.76 mm to (69.8, 24.4)
- moved SW22 4.76 mm to (69.8, 43.5)
- moved SW30 4.76 mm to (31.8, 67.3)
- moved SW32 4.76 mm to (69.8, 62.5)
- moved SW33 4.76 mm to (88.9, 67.3)
- moved SW00 4.76 mm to (31.8, 10.2)
- moved SW02 4.76 mm to (69.8, 5.40)
- moved SW03 4.76 mm to (88.9, 10.2)
- moved SW04 4.76 mm to (108.0, 14.9)
- moved SW10 4.76 mm to (31.8, 29.2)
- moved SW13 4.76 mm to (88.9, 29.2)
- moved SW20 4.76 mm to (31.8, 48.3)
- moved SW23 4.76 mm to (88.9, 48.3)
Other:
- board size 161.9 x 123.8 mm -> 161.9 x 119.1 mm
Changed lines of the file:
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@@
   )
   (module blackwing:MX_FLIP (layer F.Cu)
-    (at 88.9 62.5475)
+    (at 88.9 67.31)
     (fp_text reference SW33 (at 0 3.302) (layer F.SilkS)
       (effects (font (size 1.524 1.778) (thickness 0.254)))
@@
   )
   (module blackwing:MX_FLIP (layer F.Cu)
-    (at 69.85 57.785)
+    (at 69.85 62.5475)
     (fp_text reference SW32 (at 0 3.302) (layer F.SilkS)
       (effects (font (size 1.524 1.778) (thickness 0.254)))
@@
   )
   (module blackwing:MX_FLIP (layer F.Cu)
-    (at 31.75 62.5475)
+    (at 31.75 67.31)
     (fp_text reference SW30 (at 0 3.302) (layer F.SilkS)
       (effects (font (size 1.524 1.778) (thickness 0.254)))
@@
   )
   (module blackwing:MX_FLIP (layer F.Cu)
-    (at 88.9 43.4975)
+    (at 88.9 48.26)
     (fp_text reference SW23 (at 0 3.302) (layer F.SilkS)
       (effects (font (size 1.524 1.778) (thickness 0.254)))
@@
   )
   (module blackwing:MX_FLIP (layer F.Cu)
-    (at 31.75 5.3975)
+    (at 31.75 10.16)
     (fp_text reference SW00 (at 0 3.302) (layer F.SilkS)
       (effects (font (size 1.524 1.778) (thickness 0.254)))
@@
   )
   (module blackwing:MX_FLIP (layer F.Cu)
-    (at 50.8 3.01625)
+    (at 50.8 10.16)
     (fp_text reference SW01 (at 0 3.302) (layer F.SilkS)
       (effects (font (size 1.524 1.778) (thickness 0.254)))
@@
   )
   (module blackwing:MX_FLIP (layer F.Cu)
-    (at 69.85 0.635)
+    (at 69.85 5.3975)
     (fp_text reference SW02 (at 0 3.302) (layer F.SilkS)
       (effects (font (size 1.524 1.778) (thickness 0.254)))
@@
   )
   (module blackwing:MX_FLIP (layer F.Cu)
-    (at 88.9 5.3975)
+    (at 88.9 10.16)
     (fp_text reference SW03 (at 0 3.302) (layer F.SilkS)
       (effects (font (size 1.524 1.778) (thickness 0.254)))
@@
   )
   (module blackwing:MX_FLIP (layer F.Cu)
-    (at 107.95 10.16)
+    (at 107.95 14.9225)
     (fp_text reference SW04 (at 0 3.302) (layer F.SilkS)
       (effects (font (size 1.524 1.778) (thickness 0.254)))
@@
   )
   (module blackwing:MX_FLIP (layer F.Cu)
-    (at 31.75 24.4475)
+    (at 31.75 29.21)
     (fp_text reference SW10 (at 0 3.302) (layer F.SilkS)
       (effects (font (size 1.524 1.778) (thickness 0.254)))
@@
   )
   (module blackwing:MX_FLIP (layer F.Cu)
-    (at 69.85 19.685)
+    (at 69.85 24.4475)
     (fp_text reference SW12 (at 0 3.302) (layer F.SilkS)
       (effects (font (size 1.524 1.778) (thickness 0.254)))
@@
   )
   (module blackwing:MX_FLIP (layer F.Cu)
-    (at 88.9 24.4475)
+    (at 88.9 29.21)
     (fp_text reference SW13 (at 0 3.302) (layer F.SilkS)
       (effects (font (size 1.524 1.778) (thickness 0.254)))
@@
   )
   (module blackwing:MX_FLIP (layer F.Cu)
-    (at 31.75 43.4975)
+    (at 31.75 48.26)
     (fp_text reference SW20 (at 0 3.302) (layer F.SilkS)
       (effects (font (size 1.524 1.778) (thickness 0.254)))
@@
   )
   (module blackwing:MX_FLIP (layer F.Cu)
-    (at 69.85 38.735)
+    (at 69.85 43.4975)
     (fp_text reference SW22 (at 0 3.302) (layer F.SilkS)
       (effects (font (size 1.524 1.778) (thickness 0.254)))
@@
     )
   )
+  (gr_line (start 41.275 105.41) (end 60.325 100.6475) (layer Edge.Cuts) (width 0.15))
+  (gr_line (start 41.275 105.41) (end 22.225 114.935) (layer Edge.Cuts) (width 0.15))
   (dimension 161.925 (width 0.3) (layer F.Fab)
     (gr_text "161,925 mm" (at 84.1375 121.7975) (layer F.Fab)
@@
     (arrow2b (pts (xy 3.175 119.6975) (xy 4.301504 119.111079)))
   )
-  (dimension 123.825 (width 0.3) (layer F.Fab)
-    (gr_text "123,825 mm" (at -3.6875 53.0225 90) (layer F.Fab)
+  (dimension 119.0625 (width 0.3) (layer F.Fab)
+    (gr_text "119,062 mm" (at -3.6875 55.40375 90) (layer F.Fab)
       (effects (font (size 1.5 1.5) (thickness 0.3)))
     )
-    (feature1 (pts (xy 69.85 -8.89) (xy -2.173921 -8.89)))
+    (feature1 (pts (xy 69.85 -4.1275) (xy -2.173921 -4.1275)))
     (feature2 (pts (xy 69.85 114.935) (xy -2.173921 114.935)))
-    (crossbar (pts (xy -1.5875 114.935) (xy -1.5875 -8.89)))
-    (arrow1a (pts (xy -1.5875 -8.89) (xy -1.001079 -7.763496)))
-    (arrow1b (pts (xy -1.5875 -8.89) (xy -2.173921 -7.763496)))
+    (crossbar (pts (xy -1.5875 114.935) (xy -1.5875 -4.1275)))
+    (arrow1a (pts (xy -1.5875 -4.1275) (xy -1.001079 -3.000996)))
+    (arrow1b (pts (xy -1.5875 -4.1275) (xy -2.173921 -3.000996)))
     (arrow2a (pts (xy -1.5875 114.935) (xy -1.001079 113.808496)))
     (arrow2b (pts (xy -1.5875 114.935) (xy -2.173921 113.808496)))
   )
-  (gr_line (start 41.275 105.41) (end 60.325 100.6475) (layer Edge.Cuts) (width 0.15))
   (gr_line (start 3.175 114.935) (end 22.225 114.935) (layer Edge.Cuts) (width 0.15))
-  (gr_line (start 22.225 -4.1275) (end 60.325 -8.89) (layer Edge.Cuts) (width 0.15))
-  (gr_line (start 60.325 -8.89) (end 79.375 -8.89) (layer Edge.Cuts) (width 0.15))
-  (gr_line (start 79.375 -8.89) (end 165.1 12.54125) (layer Edge.Cuts) (width 0.15))
-  (gr_line (start 22.225 -4.1275) (end 3.175 76.835) (layer Edge.Cuts) (width 0.15))
+  (gr_line (start 22.225 0.635) (end 60.325 -4.1275) (layer Edge.Cuts) (width 0.15))
+  (gr_line (start 60.325 -4.1275) (end 79.375 -4.1275) (layer Edge.Cuts) (width 0.15))
+  (gr_line (start 79.375 -4.1275) (end 165.1 10.16) (layer Edge.Cuts) (width 0.15))
+  (gr_line (start 22.225 0.635) (end 3.175 76.835) (layer Edge.Cuts) (width 0.15))
   (gr_line (start 3.175 114.935) (end 3.175 76.835) (layer Edge.Cuts) (width 0.15))
-  (gr_line (start 41.275 105.41) (end 22.225 114.935) (layer Edge.Cuts) (width 0.15))
   (gr_line (start 165.1 100.6475) (end 60.325 100.6475) (layer Edge.Cuts) (width 0.15))
-  (gr_line (start 165.1 12.54125) (end 165.1 100.6475) (layer Edge.Cuts) (width 0.15))
+  (gr_line (start 165.1 10.16) (end 165.1 100.6475) (layer Edge.Cuts) (width 0.15))
   (segment (start 147.249729 37.4225) (end 147.249729 32.264771) (width 0.254) (layer B.Cu) (net 2) (status 1000000))
   (segment (start 147.249729 32.264771) (end 147.32 32.1945) (width 0.254) (layer B.Cu) (net 2) (status 1000000))
@@
   (segment (start 135.89 76.092934) (end 135.89 56.3365) (width 0.254) (layer F.Cu) (net 29))
   (segment (start 133.433479 78.549455) (end 135.89 76.092934) (width 0.254) (layer F.Cu) (net 29))
-  (segment (start 156.05 37.4225) (end 156.05 37.4225) (width 0.254) (layer F.Cu) (net 31))
-  (segment (start 156.05 39.2125) (end 156.05 37.4225) (width 0.254) (layer F.Cu) (net 31))
-  (via (at 156.05 37.4225) (size 0.6858) (drill 0.3302) (layers F.Cu B.Cu) (net 31))
   (segment (start 35.56 92.075) (end 35.56 93.345) (width 0.254) (layer F.Cu) (net 30))
   (segment (start 34.29 90.805) (end 35.56 92.075) (width 0.254) (layer F.Cu) (net 30))
-  (segment (start 157.15 37.4225) (end 157.15 37.4225) (width 0.254) (layer F.Cu) (net 32))
-  (via (at 157.15 37.4225) (size 0.6858) (drill 0.3302) (layers F.Cu B.Cu) (net 32))
-  (segment (start 54.61 87.3125) (end 54.61 88.5825) (width 0.254) (layer F.Cu) (net 31))
-  (segment (start 53.34 86.0425) (end 54.61 87.3125) (width 0.254) (layer F.Cu) (net 31))
-  (segment (start 157.15 39.1765) (end 157.15 37.4225) (width 0.254) (layer F.Cu) (net 32))
-  (segment (start 156.51202 39.81448) (end 157.15 39.1765) (width 0.254) (layer F.Cu) (net 32))
-  (segment (start 154.857766 39.81448) (end 156.51202 39.81448) (width 0.254) (layer F.Cu) (net 32))
-  (segment (start 137.414032 57.258214) (end 154.857766 39.81448) (width 0.254) (layer F.Cu) (net 32))
-  (segment (start 137.414031 76.724211) (end 137.414032 57.258214) (width 0.254) (layer F.Cu) (net 32))
-  (segment (start 134.064753 80.073489) (end 137.414031 76.724211) (width 0.254) (layer F.Cu) (net 32))
   (segment (start 152.75 37.4225) (end 152.75 37.4225) (width 0.254) (layer F.Cu) (net 30))
   (via (at 152.75 37.4225) (size 0.6858) (drill 0.3302) (layers F.Cu B.Cu) (net 30))
@@
   (segment (start 35.56 93.345) (end 49.847533 79.057467) (width 0.254) (layer F.Cu) (net 30))
   (segment (start 152.75 40.322498) (end 152.75 39.1765) (width 0.254) (layer F.Cu) (net 30))
+  (segment (start 156.05 37.4225) (end 156.05 37.4225) (width 0.254) (layer F.Cu) (net 31))
+  (segment (start 156.05 39.2125) (end 156.05 37.4225) (width 0.254) (layer F.Cu) (net 31))
+  (via (at 156.05 37.4225) (size 0.6858) (drill 0.3302) (layers F.Cu B.Cu) (net 31))
+  (segment (start 54.61 87.3125) (end 54.61 88.5825) (width 0.254) (layer F.Cu) (net 31))
+  (segment (start 53.34 86.0425) (end 54.61 87.3125) (width 0.254) (layer F.Cu) (net 31))
   (segment (start 53.34 86.0425) (end 54.737 84.6455) (width 0.254) (layer F.Cu) (net 31))
   (segment (start 136.906021 76.513785) (end 133.854328 79.565478) (width 0.254) (layer F.Cu) (net 31))
@@
   (segment (start 59.817022 79.565478) (end 54.737 84.6455) (width 0.254) (layer F.Cu) (net 31))
   (segment (start 59.944022 79.565478) (end 59.817022 79.565478) (width 0.254) (layer F.Cu) (net 31))
+  (segment (start 157.15 37.4225) (end 157.15 37.4225) (width 0.254) (layer F.Cu) (net 32))
+  (via (at 157.15 37.4225) (size 0.6858) (drill 0.3302) (layers F.Cu B.Cu) (net 32))
+  (segment (start 157.15 39.1765) (end 157.15 37.4225) (width 0.254) (layer F.Cu) (net 32))
+  (segment (start 156.51202 39.81448) (end 157.15 39.1765) (width 0.254) (layer F.Cu) (net 32))
+  (segment (start 154.857766 39.81448) (end 156.51202 39.81448) (width 0.254) (layer F.Cu) (net 32))
+  (segment (start 137.414032 57.258214) (end 154.857766 39.81448) (width 0.254) (layer F.Cu) (net 32))
+  (segment (start 137.414031 76.724211) (end 137.414032 57.258214) (width 0.254) (layer F.Cu) (net 32))
+  (segment (start 134.064753 80.073489) (end 137.414031 76.724211) (width 0.254) (layer F.Cu) (net 32))
   (segment (start 92.71 87.3125) (end 92.71 88.5825) (width 0.254) (layer F.Cu) (net 32))
   (segment (start 91.44 86.0425) (end 92.71 87.3125) (width 0.254) (layer F.Cu) (net 32))

Commit message: try
Connections:
- U1 pad 10: S35 -> S30
- U1 pad 14: S32 -> S34
- U1 pad 15: S30 -> S35
- U1 pad 16: S25 -> S20
- U1 pad 17: S24 -> S21
- U1 pad 18: S21 -> S22
- U1 pad 20: S22 -> S24
- U1 pad 21: S20 -> S25
- U1 pad 22: S15 -> S10
- U1 pad 23: S14 -> S11
- U1 pad 24: S11 -> S12
- U1 pad 25: S01 -> S02
- U1 pad 26: S04 -> S01
- U1 pad 28: S12 -> S14
- U1 pad 29: S10 -> S15
- U1 pad 30: S05 -> S00
- U1 pad 34: S02 -> S04
- U1 pad 35: S00 -> S05
- U1 pad 5: S31 -> S32
- U1 pad 6: S34 -> S31
- U2 pad 13: S11 -> S12
- U2 pad 14: S14 -> S11
- U2 pad 15: S15 -> S10
- U2 pad 16: S20 -> S25
- U2 pad 17: S22 -> S24
- U2 pad 19: S21 -> S22
- U2 pad 2: S00 -> S05
- U2 pad 20: S24 -> S21
- U2 pad 21: S25 -> S20
- U2 pad 22: S30 -> S35
- U2 pad 23: S32 -> S34
- U2 pad 25: S31 -> S32
- U2 pad 26: S34 -> S31
- U2 pad 27: S35 -> S30
- U2 pad 3: S02 -> S04
- U2 pad 5: S01 -> S02
- U2 pad 6: S04 -> S01
- U2 pad 7: S05 -> S00
- U2 pad 8: S10 -> S15
- U2 pad 9: S12 -> S14
Routing:
- net S32: track 92.4 -> 131.0 mm
- net S33: track 69.9 -> 98.1 mm
- net S31: track 122.1 -> 146.6 mm
- net S23: track 61.8 -> 85.5 mm
- net S22: track 83.1 -> 106.5 mm
- net S15: track 18.3 -> 40.6 mm
- net S30: track 136.7 -> 157.6 mm
- net S14: track 38.6 -> 59.1 mm
- net S21: track 101.5 -> 121.4 mm
- net S25: track 26.0 -> 44.1 mm
- net S24: track 45.7 -> 63.0 mm
- net S13: track 64.1 -> 79.0 mm
- net S35: track 40.9 -> 55.1 mm
- net S11: track 93.8 -> 107.1 mm
- net S34: track 64.9 -> 78.1 mm
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
Commit message: make outline smaller
Parts:
- moved BT2 6.33 mm to (156.8, 95.7)
- moved J1 6.22 mm to (144.9, 34.6)
- moved U1 6.22 mm to (162.6, 34.7)
- moved U2 6.22 mm to (162.6, 34.7)
- moved BT1 5.52 mm to (156.8, 47.9)
Routing:
- net S25: track 44.1 -> 24.8 mm
- net S35: track 55.1 -> 37.2 mm
- net S15: track 40.6 -> 27.4 mm
- net S24: track 63.0 -> 52.1 mm
- net S23: track 85.5 -> 74.7 mm
- net S20: track 140.2 -> 129.4 mm
- net S21: track 121.4 -> 110.6 mm
- net S34: track 78.1 -> 67.5 mm
- net S31: track 146.6 -> 136.2 mm
- net S30: track 157.6 -> 147.2 mm
- net S22: track 106.5 -> 96.1 mm
- net S10: track 126.0 -> 116.8 mm
- net S11: track 107.1 -> 98.0 mm
- net S14: track 59.1 -> 50.0 mm
- net S33: track 98.1 -> 89.3 mm
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Other:
- board size 161.9 x 119.1 mm -> 157.2 x 114.3 mm

Commit message: move key columns
Parts:
- BT1: moved to B.Cu
- BT2: moved to F.Cu
- moved BT1 12.7 mm to (144.1, 47.9)
- moved BT2 12.7 mm to (144.1, 95.7)
- moved SW22 5.68 mm to (72.4, 38.4)
- moved SW31 5.68 mm to (53.3, 62.2)
- moved SW11 5.68 mm to (53.3, 24.1)
- moved SW12 5.68 mm to (72.4, 19.4)
- moved SW30 5.68 mm to (34.3, 62.2)
- moved SW01 5.68 mm to (53.3, 5.08)
- moved SW02 5.68 mm to (72.4, 0.32)
- moved SW10 5.68 mm to (34.3, 24.1)
- moved SW21 5.68 mm to (53.3, 43.2)
- moved SW32 5.68 mm to (72.4, 57.5)
- moved SW33 5.68 mm to (91.4, 62.2)
- moved SW42 5.68 mm to (53.3, 86.0)
- moved SW40 5.68 mm to (15.2, 100.3)
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Routing:
- net GND: track 0.00 -> 1215.0 mm
- net VCC: track 79.7 -> 69.9 mm
- net S50: track 164.1 -> 165.9 mm
- removed copper zone on B.Cu, net GND
- removed copper zone on F.Cu, net GND
Other:
- net class Default: clearance 0.254 -> 0.2
- rule trace_clearance: 0.254 -> 0.2
