File: left/left.kicad_sch (KiCad schematic)
At the start: 38 parts, among them J1 Conn_01x04, J2 USB_C_Receptacle_USB2.0, SW0 SW_Push, SW1 SW_Push, SW10 SW_Push, SW11 SW_Push, SW12 SW_Push, SW13 SW_Push, SW14 SW_Push, SW15 SW_Push, SW2 SW_Push, SW20 SW_Push, SW21 SW_Push, SW22 SW_Push, SW23 SW_Push, SW24 SW_Push, SW25 SW_Push, SW3 SW_Push, SW30 SW_Push, SW31 SW_Push, SW32 SW_Push, SW33 SW_Push, SW34 SW_Push, SW35 SW_Push, SW4 SW_Push, SW40 SW_Push, SW41 SW_Push, SW42 SW_Push, SW43 SW_Push, SW44 SW_Push, SW45 SW_Push, SW5 SW_Push, SW50 SW_Push, SW6 RotaryEncoder_Switch, U1 HOLYIOT-18010-NRF52840, U2 MCP73831-3-OT

Commit message: right finished, left wip
Parts:
- removed BT1: Battery_Cell, Connector_JST:JST_PH_S2B-PH-K_1x02_P2.00mm_Horizontal, symbol Device:Battery_Cell
- removed R1: R_Small, Resistor_SMD:R_0603_1608Metric, symbol Device:R_Small
- removed U2: MCP73831-3-OT, Package_TO_SOT_SMD:SOT-23-5, symbol Battery_Management:MCP73831-3-OT
- added BT1: Battery, Battery:BatteryHolder_Keystone_2468_2xAAA, symbol Device:Battery
- added D1: D, Diode_SMD:D_SOD-123, symbol Device:D
- added H1, H2: MountingHole, MountingHole:MountingHole_2.7mm_M2.5_DIN965, symbol Mechanical:MountingHole
- added R1, R2: 5.1K, Resistor_SMD:R_0603_1608Metric, symbol Device:R
- added R3, R4: 22R, Resistor_SMD:R_0402_1005Metric, symbol Device:R
- added SW1, SW2: SW_Push, Button_Switch_SMD:SW_Push_1P1T_NO_Vertical_Wuerth_434133025816, symbol Switch:SW_Push
- SW10, SW11, SW12, SW13, SW14, SW15: footprint blackwing:MX_FLIP_5Pin -> blackwing:SW_Cherry_MX_1.00u_PCB
- SW16: renamed from SW20; footprint blackwing:MX_FLIP_5Pin -> blackwing:SW_Cherry_MX_1.00u_PCB
- SW17: renamed from SW21; footprint blackwing:MX_FLIP_5Pin -> blackwing:SW_Cherry_MX_1.00u_PCB
- SW18: renamed from SW22; footprint blackwing:MX_FLIP_5Pin -> blackwing:SW_Cherry_MX_1.00u_PCB
- SW19: renamed from SW23; footprint blackwing:MX_FLIP_5Pin -> blackwing:SW_Cherry_MX_1.00u_PCB
- SW20: renamed from SW24; footprint blackwing:MX_FLIP_5Pin -> blackwing:SW_Cherry_MX_1.00u_PCB
- SW21: renamed from SW25; footprint blackwing:MX_FLIP_5Pin -> blackwing:SW_Cherry_MX_1.00u_PCB
- SW22: renamed from SW30; footprint blackwing:MX_FLIP_5Pin -> blackwing:SW_Cherry_MX_1.00u_PCB
- SW23: renamed from SW31; footprint blackwing:MX_FLIP_5Pin -> blackwing:SW_Cherry_MX_1.00u_PCB
- SW24: renamed from SW32; footprint blackwing:MX_FLIP_5Pin -> blackwing:SW_Cherry_MX_1.00u_PCB
- SW25: renamed from SW33; footprint blackwing:MX_FLIP_5Pin -> blackwing:SW_Cherry_MX_1.00u_PCB
- SW26: renamed from SW34; footprint blackwing:MX_FLIP_5Pin -> blackwing:SW_Cherry_MX_1.00u_PCB
- SW27: renamed from SW35; footprint blackwing:MX_FLIP_5Pin -> blackwing:SW_Cherry_MX_1.00u_PCB
- SW28: renamed from SW40; footprint blackwing:MX_FLIP_5Pin -> blackwing:SW_Cherry_MX_1.00u_PCB
- SW29: renamed from SW41; footprint blackwing:MX_FLIP_5Pin -> blackwing:SW_Cherry_MX_1.00u_PCB
- SW30: renamed from SW42; footprint blackwing:MX_FLIP_5Pin -> blackwing:SW_Cherry_MX_1.00u_PCB
- SW31: renamed from SW43; footprint blackwing:MX_FLIP_5Pin_1.25u -> blackwing:SW_Cherry_MX_1.25u_PCB
- SW32: renamed from SW44; footprint blackwing:MX_FLIP_5Pin -> blackwing:SW_Cherry_MX_1.00u_PCB
- SW33: renamed from SW45; footprint blackwing:MX_FLIP_5Pin_1.25u -> blackwing:SW_Cherry_MX_1.25u_PCB
- SW34: renamed from SW50; footprint blackwing:MX_FLIP_5Pin -> blackwing:SW_Cherry_MX_1.75u_PCB
- SW4: renamed from SW0; footprint blackwing:MX_FLIP_5Pin -> blackwing:SW_Cherry_MX_1.00u_PCB
- SW5: renamed from SW1; footprint blackwing:MX_FLIP_5Pin -> blackwing:SW_Cherry_MX_1.00u_PCB
- SW6: renamed from SW2; footprint blackwing:MX_FLIP_5Pin -> blackwing:SW_Cherry_MX_1.00u_PCB
- SW7: renamed from SW3; footprint blackwing:MX_FLIP_5Pin -> blackwing:SW_Cherry_MX_1.00u_PCB
- SW8: renamed from SW4; footprint blackwing:MX_FLIP_5Pin -> blackwing:SW_Cherry_MX_1.00u_PCB
- SW9: renamed from SW5; footprint blackwing:MX_FLIP_5Pin -> blackwing:SW_Cherry_MX_1.00u_PCB
- renumbered J2 to J1, J1 to J2, SW6 to SW3
Connections:
- net +BATT is gone; now on net VCC: U1.14 (VDD-nRF)
- net D+: now also R4.2; no longer J1.A6 (D+), J1.B6 (D+)
- net D-: now also R3.2; no longer J1.A7 (D-), J1.B7 (D-)
- net GND: now also SW10.2, SW11.2, SW12.2, SW13.2, SW14.2, SW15.2, SW16.2, SW17.2, SW18.2, SW19.2, SW20.2, SW21.2, SW22.2, SW23.2, SW24.2, SW25.2, SW26.2, SW27.2, SW28.2, SW29.2, SW30.2, SW31.2, SW32.2, SW33.2, SW34.2, SW4.2, SW5.2, SW6.2, SW7.2, SW8.2, SW9.2, BT1.2 (-), R1.1, R2.1, SW1.2, SW2.2; no longer SW10.1, SW11.1, SW12.1, SW13.1, SW14.1, SW15.1, SW16.1, SW17.1, SW18.1, SW19.1, SW20.1, SW21.1, SW22.1, SW23.1, SW24.1, SW25.1, SW26.1, SW27.1, SW28.1, SW29.1, SW30.1, SW31.1, SW32.1, SW33.1, SW34.1, SW4.1, SW5.1, SW6.1, SW7.1, SW8.1, SW9.1
- net ROT_A: now also U1.2 (P1.11); no longer U1.7 (P0.02)
- net ROT_B: now also U1.3 (P1.10); no longer U1.8 (P0.28)
- net ROT_Switch: now also U1.4 (P1.13); no longer U1.9 (P0.29)
- net S00: now also SW4.1, U1.11 (P0.31); no longer SW4.2, U1.36 (P0.10)
- net S01: now also SW5.1, U1.20 (P0.19); no longer SW5.2, U1.35 (P0.09)
- net S02: now also SW6.1, U1.38 (P1.14); no longer SW6.2, U1.34 (P1.06)
- net S03: now also SW7.1, U1.29 (P1.01); no longer SW7.2, U1.33 (P1.04)
- net S04: now also SW8.1, U1.55 (P0.16); no longer SW8.2, U1.29 (P1.01)
- net S05: now also SW9.1, U1.47 (P1.07); no longer SW9.2, U1.30 (P1.02)
- net S10: now also SW10.1, U1.12 (P0.04); no longer SW10.2, U1.28 (P1.03)
- net S11: now also SW11.1, U1.19 (P0.21); no longer SW11.2, U1.27 (P1.00)
- net S12: now also SW12.1, U1.39 (P1.12); no longer SW12.2, U1.26 (P0.22)
- net S13: now also SW13.1, U1.28 (P1.03); no longer SW13.2, U1.11 (P0.31)
- net S14: now also SW14.1, U1.54 (P0.13); no longer SW14.2, U1.13 (P0.05)
- net S15: now also SW15.1, U1.48 (P1.05); no longer SW15.2, U1.10 (P0.30)
- net S20: now also SW16.1, U1.13 (P0.05); no longer SW16.2, U1.47 (P1.07)
- net S21: now also SW17.1, U1.46 (P0.26); no longer SW17.2, U1.48 (P1.05)
- net S22: now also SW18.1, U1.40 (P0.25); no longer SW18.2, U1.49 (P0.24)
- net S23: now also SW19.1, U1.27 (P1.00); no longer SW19.2, U1.45 (P0.06)
- net S24: now also SW20.1, U1.53 (P0.14); no longer SW20.2, U1.46 (P0.26)
- net S25: now also SW21.1, U1.49 (P0.24); no longer SW21.2, U1.12 (P0.04)
- net S30: now also SW22.1, U1.15 (P0.07); no longer SW22.2, U1.50 (P0.20)
- net S31: now also SW23.1, U1.45 (P0.06); no longer SW23.2, U1.51 (P0.17)
- net S32: now also SW24.1, U1.41 (P0.11); no longer SW24.2, U1.52 (P0.15)
- net S33: now also SW25.1, U1.26 (P0.22); no longer SW25.2, U1.42 (P1.08)
- net S34: now also SW26.1, U1.52 (P0.15); no longer SW26.2, U1.43 (P0.27)
- net S35: now also SW27.1, U1.50 (P0.20); no longer SW27.2, U1.44 (P0.08)
- net S40: now also SW28.1, U1.17 (P0.12); no longer SW28.2, U1.54 (P0.13)
- net S41: now also SW29.1, U1.18 (P0.23); no longer SW29.2, U1.55 (P0.16)
- net S42: now also SW30.1, U1.44 (P0.08); no longer SW30.2, U1.38 (P1.14)
- net S43: now also SW31.1, U1.43 (P0.27); no longer SW31.2, U1.39 (P1.12)
- net S44: now also SW32.1, U1.42 (P1.08); no longer SW32.2, U1.40 (P0.25)
- net S45: now also SW33.1, U1.51 (P0.17); no longer SW33.2, U1.41 (P0.11)
- net S50: now also SW34.1, U1.16 (P1.09); no longer SW34.2, U1.53 (P0.14)
- net VCC: now also D1.1 (K)
- net at J1.A5 (CC1): now also R2.2
- net at J1.B5 (CC2): now also R1.2
- net RESET: now reaches U1.21 (P0.18)
- net RESET: now also SW1.1
- new net: J1.A7 (D-), J1.B7 (D-), R3.1
- new net: BT1.1 (+), D1.2 (A)
- new net: J1.A6 (D+), J1.B6 (D+), R4.1
- new net BOOT: SW2.1, U1.36 (P0.10)
