File: left/left.kicad_pcb (KiCad board)
At the start: 2 copper layers, 143.8 x 147.7 mm, 45 parts, among them J1 USB_C_Receptacle_USB2.0, J2 Conn_01x04, SW1 SW_Push, SW10 SW_Push, SW11 SW_Push, SW12 SW_Push, SW13 SW_Push, SW14 SW_Push, SW15 SW_Push, SW16 SW_Push, SW17 SW_Push, SW18 SW_Push, SW19 SW_Push, SW2 SW_Push, SW20 SW_Push, SW21 SW_Push, SW22 SW_Push, SW23 SW_Push, SW24 SW_Push, SW25 SW_Push, SW26 SW_Push, SW27 SW_Push, SW28 SW_Push, SW29 SW_Push, SW3 RotaryEncoder_Switch, SW30 SW_Push, SW31 SW_Push, SW32 SW_Push, SW33 SW_Push, SW34 SW_Push, SW4 SW_Push, SW5 SW_Push, SW6 SW_Push, SW7 SW_Push, SW8 SW_Push, SW9 SW_Push, U1 HOLYIOT-18010-NRF52840

Commit message: right finished, left wip
Parts:
- BT1, D1, H1, H2, J1, J2, R1, R2, R3, R4, SW1, SW10, SW11, SW12, SW13, SW14, SW15, SW16, SW17, SW18, SW19, SW2, SW20, SW21, SW22, SW23, SW24, SW25, SW26, SW27, SW3, SW30, SW31, SW32, SW33, SW4, SW5, SW6, SW7, SW8, SW9, U1: moved to B.Cu
- moved U1 13.5 mm to (112.4, 19.0), turned to 180 degrees
- moved BT1 12.7 mm to (143.0, 38.1)
- moved J1 5.95 mm to (85.9, 45.5), turned to 90 degrees
- moved SW12 5.08 mm to (129.9, 74.0), turned to 0 degrees
- moved SW13 5.08 mm to (148.9, 78.7), turned to 0 degrees
- moved SW14 5.08 mm to (167.9, 83.5), turned to 0 degrees
- moved SW15 5.08 mm to (186.9, 83.5), turned to 0 degrees
- moved SW19 5.08 mm to (148.9, 97.7), turned to 0 degrees
- moved SW20 5.08 mm to (167.9, 102.5), turned to 0 degrees
- moved SW25 5.08 mm to (148.9, 116.7), turned to 0 degrees
- moved SW31 5.08 mm to (141.8, 140.5), turned to 0 degrees
- moved SW33 5.08 mm to (184.6, 140.5), turned to 0 degrees
- moved SW8 5.08 mm to (167.9, 64.5), turned to 0 degrees
- moved SW10 5.08 mm to (91.9, 78.7), turned to 0 degrees
- moved SW11 5.08 mm to (110.9, 78.7), turned to 0 degrees
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Routing:
- net S45: track 160.4 -> 0.00 mm
- net S35: track 143.3 -> 0.00 mm
- net S34: track 141.9 -> 0.00 mm
- net S44: track 139.7 -> 0.00 mm
- net S40: track 131.9 -> 0.00 mm
- net S43: track 126.1 -> 0.00 mm
- net S25: track 125.2 -> 0.00 mm
- net S24: track 121.6 -> 0.00 mm
- net S50: track 116.8 -> 0.00 mm
- net S42: track 116.7 -> 0.00 mm
- net S41: track 113.2 -> 0.00 mm
- net S15: track 107.1 -> 0.00 mm
- net S14: track 101.3 -> 0.00 mm
- net S33: track 99.0 -> 0.00 mm
- net S31: track 95.6 -> 0.00 mm
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
Commit message: finish left
Parts:
- added H3: MountingHole, MountingHole:MountingHole_2.7mm_M2.5_DIN965, F.Cu at (127.4, 26.1)
- added J3: Conn_01x06, Connector_PinHeader_2.54mm:PinHeader_1x06_P2.54mm_Vertical, B.Cu at (121.3, 118.5)
- SW28, SW29, SW34: moved to B.Cu
- moved BT1 54.4 mm to (193.9, 19.0), turned to 180 degrees
- moved R3 13.0 mm to (101.2, 39.6), turned to 90 degrees
- moved R4 11.1 mm to (99.7, 39.6), turned to 90 degrees
- moved SW28 5.08 mm to (83.1, 154.8), turned to 48 degrees
- moved SW34 5.08 mm to (73.8, 136.8), turned to 48 degrees
- moved SW29 5.08 mm to (100.2, 143.7), turned to 24 degrees
- moved SW1 4.75 mm to (117.9, 26.1), turned to -90 degrees
- moved J2 4.75 mm to (132.1, 24.7)
- moved SW2 4.70 mm to (122.6, 26.1)
- moved D1 2.97 mm to (137.5, 26.4), turned to -90 degrees
- moved H2 0.36 mm to (115.3, 42.5)
- moved H1 0.25 mm to (184.4, 47.3)
Connections:
- SW3 pad S1: ROT_Switch -> GND
- SW3 pad S2: GND -> ROT_Switch
- U1 pad 11: S00 -> S04
- U1 pad 12: S10 -> S03
- U1 pad 13: S20 -> S02
- U1 pad 15: S30 -> S01
- U1 pad 16: S50 -> S11
- U1 pad 17: S40 -> S21
- U1 pad 19: S11 -> S40
- U1 pad 2: ROT_A -> BOOT
- U1 pad 20: S01 -> S50
- U1 pad 26: S33 -> S31
- U1 pad 27: S23 -> S30
- U1 pad 28: S13 -> S20
- U1 pad 29: S03 -> S10
- U1 pad 3: ROT_B -> unconnected-(U1-Pad3)
- U1 pad 30: unconnected-(U1-Pad30) -> S00
- U1 pad 34: unconnected-(U1-Pad34) -> ROT_Switch
- U1 pad 35: unconnected-(U1-Pad35) -> ROT_A
- U1 pad 36: BOOT -> ROT_B
- U1 pad 38: S02 -> S05
- U1 pad 39: S12 -> S15
- U1 pad 4: ROT_Switch -> unconnected-(U1-Pad4)
- U1 pad 40: S22 -> S25
- U1 pad 41: S32 -> S35
- U1 pad 42: S44 -> S45
- U1 pad 43: S43 -> S44
- U1 pad 44: S42 -> S34
- U1 pad 45: S31 -> S24
- U1 pad 46: S21 -> S14
- U1 pad 47: S05 -> S13
- U1 pad 48: S15 -> S23
- U1 pad 49: S25 -> S33
- U1 pad 50: S35 -> S43
- U1 pad 51: S45 -> S42
- U1 pad 52: S34 -> S60
- U1 pad 53: S24 -> S32
- U1 pad 54: S14 -> S22
- U1 pad 55: S04 -> S12
Routing:
- net S45: track 0.00 -> 166.5 mm
- net S44: track 0.00 -> 161.7 mm
- net S40: track 0.00 -> 158.4 mm
- net S50: track 0.00 -> 152.0 mm
- net S35: track 0.00 -> 149.3 mm
- net S42: track 0.00 -> 145.3 mm
- net S41: track 0.00 -> 145.2 mm
- net VCC: track 0.00 -> 142.7 mm, vias 0 -> 1
- net S43: track 0.00 -> 140.5 mm
- net S34: track 0.00 -> 139.4 mm
- net S25: track 0.00 -> 131.2 mm
- net S33: track 0.00 -> 124.3 mm
- net S24: track 0.00 -> 119.1 mm
- net S60: track 0.00 -> 116.3 mm
- net S15: track 0.00 -> 113.1 mm
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Other:
- board text added: "GND"
- board text added: "P0.15"
- board text added: "P0.19"
- board text added: "P0.21"
- board text added: "P0.23"
- board text added: "VCC"
