File: right/blackwing.kicad_sch (KiCad schematic)
At the start: 50 parts, among them J1 USB_C_Receptacle_USB2.0, J2 Conn_01x04, SW1 SW_Push, SW10 SW_Push, SW11 SW_Push, SW12 SW_Push, SW13 SW_Push, SW14 SW_Push, SW15 SW_Push, SW16 SW_Push, SW17 SW_Push, SW18 SW_Push, SW19 SW_Push, SW2 SW_Push, SW20 SW_Push, SW21 SW_Push, SW22 SW_Push, SW23 SW_Push, SW24 SW_Push, SW25 SW_Push, SW26 SW_Push, SW27 SW_Push, SW28 SW_Push, SW29 SW_Push, SW3 RotaryEncoder_Switch, SW30 SW_Push, SW31 SW_Push, SW32 SW_Push, SW33 SW_Push, SW34 SW_Push, SW35 SW_SPDT, SW4 SW_Push, SW5 SW_Push, SW6 SW_Push, SW7 SW_Push, SW8 SW_Push, SW9 SW_Push, U1 HOLYIOT-18010-NRF52840, U2 MCP73831-2-OT

Commit message: right finished, left wip
Parts:
- removed BT1: Battery_Cell, Connector_JST:JST_PH_S2B-PH-K_1x02_P2.00mm_Horizontal, symbol Device:Battery_Cell
- removed C1, C2: 4.7µF, Capacitor_SMD:C_0603_1608Metric, symbol Device:C
- removed D1: LED, LED_SMD:LED_0603_1608Metric, symbol Device:LED_Small
- removed R1: 10K, Resistor_SMD:R_0603_1608Metric, symbol Device:R_Small
- removed R6: R, Resistor_SMD:R_0603_1608Metric, symbol Device:R_Small
- removed SW35: SW_SPDT, Button_Switch_THT:SW_CuK_OS102011MA1QN1_SPDT_Angled, symbol Switch:SW_SPDT
- removed U2: MCP73831-2-OT, Package_TO_SOT_SMD:SOT-23-5, symbol Battery_Management:MCP73831-2-OT
- added D1: D, Diode_SMD:D_SOD-123, symbol Device:D
- added H1, H2: MountingHole, MountingHole:MountingHole_2.7mm_M2.5_DIN965, symbol Mechanical:MountingHole
- SW10, SW11, SW12, SW13, SW14, SW15, SW16, SW17, SW18, SW19, SW20, SW21, SW22, SW23, SW24, SW25, SW26, SW27, SW28, SW29, SW30, SW32, SW4, SW5, SW6, SW7, SW8, SW9: footprint Button_Switch_Keyboard:SW_Cherry_MX_1.00u_PCB -> blackwing:SW_Cherry_MX_1.00u_PCB
- SW31, SW33: footprint Button_Switch_Keyboard:SW_Cherry_MX_1.25u_PCB -> blackwing:SW_Cherry_MX_1.25u_PCB
- SW34: footprint Button_Switch_Keyboard:SW_Cherry_MX_1.50u_PCB -> blackwing:SW_Cherry_MX_1.75u_PCB
- renumbered BT2 to BT1, R2 to R1, R3 to R2, R4 to R3, R5 to R4
Connections:
- net BOOT: now also U1.36 (P0.10); no longer U1.19 (P0.21)
- net RESET: now also U1.21 (P0.18); no longer U1.20 (P0.19)
- net ROT_A: now also U1.2 (P1.11); no longer U1.28 (P1.03)
- net ROT_B: now also U1.3 (P1.10); no longer U1.29 (P1.01)
- net ROT_Switch: now also U1.4 (P1.13); no longer U1.21 (P0.18)
- net S00: now also U1.11 (P0.31); no longer U1.2 (P1.11)
- net S01: now also U1.20 (P0.19); no longer U1.3 (P1.10)
- net S02: now also U1.38 (P1.14); no longer U1.4 (P1.13)
- net S03: now also U1.29 (P1.01); no longer U1.5 (P1.15)
- net S04: now also U1.55 (P0.16); no longer U1.6 (P0.03)
- net S05: now also U1.47 (P1.07); no longer U1.7 (P0.02)
- net S10: now also U1.12 (P0.04); no longer U1.8 (P0.28)
- net S11: now also U1.19 (P0.21); no longer U1.9 (P0.29)
- net S12: now also U1.39 (P1.12); no longer U1.10 (P0.30)
- net S13: now also U1.28 (P1.03); no longer U1.11 (P0.31)
- net S14: now also U1.54 (P0.13); no longer U1.12 (P0.04)
- net S15: now also U1.48 (P1.05); no longer U1.13 (P0.05)
- net S20: now also U1.13 (P0.05); no longer U1.38 (P1.14)
- net S21: now also U1.46 (P0.26); no longer U1.39 (P1.12)
- net S23: now also U1.27 (P1.00); no longer U1.48 (P1.05)
- net S24: now also U1.53 (P0.14); no longer U1.47 (P1.07)
- net S25: now also U1.49 (P0.24); no longer U1.26 (P0.22)
- net S30: now also U1.15 (P0.07); no longer U1.41 (P0.11)
- net S31: now also U1.45 (P0.06); no longer U1.42 (P1.08)
- net S32: now also U1.41 (P0.11); no longer U1.43 (P0.27)
- net S33: now also U1.26 (P0.22); no longer U1.51 (P0.17)
- net S34: now also U1.52 (P0.15); no longer U1.50 (P0.20)
- net S35: now also U1.50 (P0.20); no longer U1.49 (P0.24)
- net S40: now also U1.17 (P0.12); no longer U1.45 (P0.06)
- net S41: now also U1.18 (P0.23); no longer U1.46 (P0.26)
- net S42: now also U1.44 (P0.08); no longer U1.55 (P0.16)
- net S43: now also U1.43 (P0.27); no longer U1.54 (P0.13)
- net S44: now also U1.42 (P1.08); no longer U1.53 (P0.14)
- net S45: now also U1.51 (P0.17); no longer U1.52 (P0.15)
- net S50: now also U1.16 (P1.09); no longer U1.44 (P0.08)
- net VCC: now also D1.1 (K)
- net +BATT: no longer names the net of BT1.1 (+)
- net +BATT: now also D1.2 (A)
