File: right/right.kicad_sch (KiCad schematic)
At the start: 47 parts, among them J1 USB_C_Receptacle_USB2.0, J2 Conn_01x04, J3 Conn_01x06, SW1 SW_Push, SW10 SW_Push, SW11 SW_Push, SW12 SW_Push, SW13 SW_Push, SW14 SW_Push, SW15 SW_Push, SW16 SW_Push, SW17 SW_Push, SW18 SW_Push, SW19 SW_Push, SW2 SW_Push, SW20 SW_Push, SW21 SW_Push, SW22 SW_Push, SW23 SW_Push, SW24 SW_Push, SW25 SW_Push, SW26 SW_Push, SW27 SW_Push, SW28 SW_Push, SW29 SW_Push, SW3 RotaryEncoder_Switch, SW30 SW_Push, SW31 SW_Push, SW32 SW_Push, SW33 SW_Push, SW34 SW_Push, SW4 SW_Push, SW5 SW_Push, SW6 SW_Push, SW7 SW_Push, SW8 SW_Push, SW9 SW_Push, U1 HOLYIOT-18010-NRF52840

Commit message: finish left
Parts:
- removed J3: Conn_01x06, Connector_PinHeader_2.54mm:PinHeader_1x06_P2.54mm_Vertical, symbol Connector_Generic:Conn_01x06
Connections:
- net S60 is gone; now on net S34: U1.52 (P0.15)
- net BOOT: now also U1.36 (P0.10); no longer U1.2 (P1.11)
- net GND: now also SW3.S2; no longer SW3.S1
- net ROT_A: now also U1.2 (P1.11); no longer U1.35 (P0.09)
- net ROT_B: now also U1.3 (P1.10); no longer U1.36 (P0.10)
- net ROT_Switch: now also SW3.S1, U1.4 (P1.13); no longer SW3.S2, U1.34 (P1.06)
- net S00: now also U1.11 (P0.31); no longer U1.30 (P1.02)
- net S01: now also U1.20 (P0.19); no longer U1.15 (P0.07)
- net S02: now also U1.38 (P1.14); no longer U1.13 (P0.05)
- net S03: now also U1.29 (P1.01); no longer U1.12 (P0.04)
- net S04: now also U1.55 (P0.16); no longer U1.11 (P0.31)
- net S05: now also U1.47 (P1.07); no longer U1.38 (P1.14)
- net S10: now also U1.12 (P0.04); no longer U1.29 (P1.01)
- net S11: now also U1.19 (P0.21); no longer U1.16 (P1.09)
- net S12: now also U1.39 (P1.12); no longer U1.55 (P0.16)
- net S13: now also U1.28 (P1.03); no longer U1.47 (P1.07)
- net S14: now also U1.54 (P0.13); no longer U1.46 (P0.26)
- net S15: now also U1.48 (P1.05); no longer U1.39 (P1.12)
- net S20: now also U1.13 (P0.05); no longer U1.28 (P1.03)
- net S21: now also U1.46 (P0.26); no longer U1.17 (P0.12)
- net S22: now also U1.40 (P0.25); no longer U1.54 (P0.13)
- net S23: now also U1.27 (P1.00); no longer U1.48 (P1.05)
- net S24: now also U1.53 (P0.14); no longer U1.45 (P0.06)
- net S25: now also U1.49 (P0.24); no longer U1.40 (P0.25)
- net S30: now also U1.15 (P0.07); no longer U1.27 (P1.00)
- net S31: now also U1.45 (P0.06); no longer U1.26 (P0.22)
- net S32: now also U1.41 (P0.11); no longer U1.53 (P0.14)
- net S33: now also U1.26 (P0.22); no longer U1.49 (P0.24)
- net S34: no longer U1.44 (P0.08)
- net S35: now also U1.50 (P0.20); no longer U1.41 (P0.11)
- net S40: now also U1.17 (P0.12); no longer U1.19 (P0.21)
- net S42: now also U1.44 (P0.08); no longer U1.51 (P0.17)
- net S43: now also U1.43 (P0.27); no longer U1.50 (P0.20)
- net S44: now also U1.42 (P1.08); no longer U1.43 (P0.27)
- net S45: now also U1.51 (P0.17); no longer U1.42 (P1.08)
- net S50: now also U1.16 (P1.09); no longer U1.20 (P0.19)
- no-connect marks 9 -> 12
