File: right/right.kicad_pcb (KiCad board)
At the start: 2 copper layers, 143.8 x 147.7 mm, 46 parts, among them J1 USB_C_Receptacle_USB2.0, J2 Conn_01x04, SW1 SW_Push, SW10 SW_Push, SW11 SW_Push, SW12 SW_Push, SW13 SW_Push, SW14 SW_Push, SW15 SW_Push, SW16 SW_Push, SW17 SW_Push, SW18 SW_Push, SW19 SW_Push, SW2 SW_Push, SW20 SW_Push, SW21 SW_Push, SW22 SW_Push, SW23 SW_Push, SW24 SW_Push, SW25 SW_Push, SW26 SW_Push, SW27 SW_Push, SW28 SW_Push, SW29 SW_Push, SW3 RotaryEncoder_Switch, SW30 SW_Push, SW31 SW_Push, SW32 SW_Push, SW33 SW_Push, SW34 SW_Push, SW4 SW_Push, SW5 SW_Push, SW6 SW_Push, SW7 SW_Push, SW8 SW_Push, SW9 SW_Push, U1 HOLYIOT-18010-NRF52840

Commit message: update footprint of rf module
Parts:
- moved BT1 51.3 mm to (143.0, 25.5)
- moved R3 0.12 mm to (88.9, 43.5)
Routing:
- net VCC: track 48.5 -> 50.7 mm
- net S05: vias 0 -> 1
- net S44: vias 0 -> 1
- net S43: vias 0 -> 1
- net S42: vias 0 -> 1
- net S31: vias 0 -> 1
- net S24: vias 0 -> 1
- net S15: vias 0 -> 1
- net S45: vias 0 -> 1
- net S35: vias 0 -> 1
- net S34: vias 0 -> 1
- net S32: vias 0 -> 1
- net S25: vias 0 -> 1
- net S22: vias 0 -> 1
- net S21: vias 0 -> 1
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
Commit message: minor fixes
Routing:
- net S02: track 42.6 -> 40.9 mm
